File: PCB/Main Board Ver 0.2/Schematic Ver 0.3.kicad_pcb (KiCad board)
At the start: 2 copper layers, 86.7 x 66.9 mm, 23 parts, among them P1 CONN_01X07, P10 CONN_01X07, P11 LCD_Interface, P12 CONN_10, P13 Start Buttons, P14 CONN_1, P15 CONN_1, P16 CONN_1, P17 CONN_1, P2 CONN_01X07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

Commit message: Added Plots of boards, now ready to be ordered
Parts:
- added P18: CONN_4, PIN_ARRAY_4x1, F.Cu at (219.7, 179.3)
Connections:
- P12 pad 6: N-0000012 (its old number) -> (no net)
- P12 pad 7: N-0000014 (its old number) -> (no net)
- P12 pad 8: N-0000015 (its old number) -> (no net)
- P12 pad 9: N-0000016 (its old number) -> (no net)
- P4 pad 1: N-0000016 (its old number) -> N-0000024
- P4 pad 2: N-0000015 (its old number) -> N-0000023
- P4 pad 3: N-0000014 (its old number) -> N-0000017
- P4 pad 4: N-0000012 (its old number) -> N-0000022
Routing:
- net N-0000016 (its old number): track 15.2 -> 0.00 mm
- net N-0000015 (its old number): track 15.2 -> 0.00 mm
- net N-0000014 (its old number): track 15.2 -> 0.00 mm
- net N-0000012 (its old number): track 15.2 -> 0.00 mm
- net N-0000024: track 0.00 -> 7.87 mm
- net N-0000023: track 0.00 -> 7.87 mm
- net N-0000022: track 0.00 -> 7.87 mm
- net N-0000017: track 0.00 -> 7.87 mm
