File: PCB/Main Board Ver 0.2/Schematic Ver 0.3.sch (KiCad schematic (older format))
At the start: 23 parts, among them P1 CONN_01X07, P10 CONN_01X07, P11 LCD_Interface, P12 CONN_10, P13 Start Buttons, P14 CONN_1, P15 CONN_1, P16 CONN_1, P17 CONN_1, P2 CONN_01X07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

Commit message: Added Plots of boards, now ready to be ordered
Parts:
- added P18: CONN_4, ~, symbol CONN_4
Connections:
- net at P4.1: now also P18.4 (P4); no longer P12.9 (P9)
- net at P4.2: now also P18.3 (P3); no longer P12.8 (P8)
- net at P4.3: now also P18.2 (P2); no longer P12.7 (P7)
- net at P4.4: now also P18.1 (P1); no longer P12.6 (P6)
- no-connect marks 13 -> 17
Changed lines of the file:
@@
 Sheet 1 1
 Title ""
-Date "29 nov 2016"
+Date "22 dec 2016"
 Rev ""
 Comp ""
@@
 $EndComp
 Wire Wire Line
-	4400 2600 5200 2600
-Wire Wire Line
-	4400 2700 5200 2700
-Wire Wire Line
-	4400 2800 5200 2800
-Wire Wire Line
-	4400 2900 5200 2900
-Wire Wire Line
 	4400 3000 5200 3000
 Wire Wire Line
@@
 	0    1    1    0
 $EndComp
+$Comp
+L CONN_4 P18
+U 1 1 585B20A8
+P 4750 2750
+F 0 "P18" V 4700 2750 50  0000 C CNN
+F 1 "CONN_4" V 4800 2750 50  0000 C CNN
+F 2 "~" H 4750 2750 60  0000 C CNN
+F 3 "~" H 4750 2750 60  0000 C CNN
+	1    4750 2750
+	-1   0    0    1
+$EndComp
+Wire Wire Line
+	5100 2600 5200 2600
+Wire Wire Line
+	5200 2700 5100 2700
+Wire Wire Line
+	5100 2800 5200 2800
+Wire Wire Line
+	5200 2900 5100 2900
+NoConn ~ 4400 2600
+NoConn ~ 4400 2700
+NoConn ~ 4400 2800
+NoConn ~ 4400 2900
 $EndSCHEMATC
